Commit message: SMB, cleaned up file structure.

File: urdf/usafabot.urdf (robot description, URDF)
Before this commit: robot usafabot, 7 links, 6 joints
Links:
- link base_link: geometry visual mesh filename=package://usafabot/meshes/bottom_chassis.stl scale=.001 .001 .001
- link left_wheel: geometry visual mesh filename=package://usafabot/meshes/rviz_wheel2.stl scale=.001 .001 .001
- link right_wheel: geometry visual mesh filename=package://usafabot/meshes/rviz_wheel1.stl scale=.001 .001 .001
- link top_chassis: geometry visual mesh filename=package://usafabot/meshes/top_chassis.stl scale=.001 .001 .001

Commit message: SMB, 2 Aug 2021, updated urdf base_link offset.

File: urdf/usafabot.urdf (robot description, URDF)
Before this commit: robot usafabot, 7 links, 6 joints
Joints:
- joint base_joint: origin xyz=0.0 0.0 0.035 rpy=0 0 0 -> xyz=0.0 0.0 0.005 rpy=0 0 0

Commit message: SMB, updated code.

File: urdf/usafabot.urdf (robot description, URDF)
Before this commit: robot usafabot, 7 links, 6 joints
Links:
- added link roadrunner; visual box size=.1 .04 0.05
Joints:
- added joint joint_roadrunner: type fixed, parent roadrunner, child base_footprint, origin xyz=0.0 0.0 -0.115 rpy=0 0 0
