Commit message: SMB, fixed usafabot so it will work for multiple robots. Adds hostname to TF and topics. Also moved roadrunner code to usafabot.

File: urdf/usafabot.xacro (robot description, xacro)
@@ -1,8 +1,10 @@
 <?xml version='1.0'?>
-<robot name="usafabot">
+<robot name="$(env HOSTNAME)" xmlns:xacro="http://www.ros.org/wiki/xacro">
+<xacro:arg name="robot_name" default=""/>
+<xacro:property name="namespace" value="$(arg robot_namespace)" />
 <!-- * * * Link Definitions * * * -->
-        <link name="base_footprint"/>
-        <link name="imu_link"/>
-	<link name="base_link">
+        <link name="$(arg robot_name)_base_footprint"/>
+        <link name="$(arg robot_name)_imu_link"/>
+	<link name="$(arg robot_name)_base_link">
 	<visual>
 	  <origin xyz="0 0 0.005" rpy="1.5708 0 1.5708" />
@@ -15,5 +17,5 @@
 	</visual>
 	</link>
-	<link name="top_chassis">
+	<link name="$(arg robot_name)_top_chassis">
 	<visual>
 	  <origin xyz="0 0 0" rpy="0 0 1.5708" />
@@ -26,5 +28,5 @@
 	</visual>
 	</link>
-	<link name="right_wheel">
+	<link name="$(arg robot_name)_right_wheel">
 	<visual>
 	  <origin xyz="0 0 0" rpy="0 0 1.5708" />
@@ -37,5 +39,5 @@
 	</visual>
 	</link>
-	<link name="left_wheel">
+	<link name="$(arg robot_name)_left_wheel">
 	<visual>
 	  <origin xyz="0 0 0" rpy="0 3.1415 1.5708" />
@@ -48,5 +50,5 @@
 	</visual>
 	</link>
-	<link name="laser">
+	<link name="$(arg robot_name)_laser">
 	<visual>
 	  <origin xyz="0 0 0" rpy="0 0 0" />
@@ -59,5 +61,5 @@
 	</visual>
 	</link>
-	<link name="roadrunner">
+	<link name="$(arg robot_name)_roadrunner">
 	<visual>
 	  <origin xyz="0 0 0" rpy="0 0 0" />
@@ -71,38 +73,38 @@
 	</link>
 	<!-- * * * Joint Definitions * * * -->
-        <joint name="base_joint" type="fixed">
-                <parent link="base_footprint"/>
-		<child link ="base_link"/>
+        <joint name="$(arg robot_name)_base_joint" type="fixed">
+                <parent link="$(arg robot_name)_base_footprint"/>
+		<child link ="$(arg robot_name)_base_link"/>
 		<origin xyz="0.0 0.0 0.005" rpy="0 0 0"/>
 	</joint>
-        <joint name="joint_top_chassis" type="fixed">
-		<parent link="base_link"/>
-		<child link="top_chassis"/>
+        <joint name="$(arg robot_name)_joint_top_chassis" type="fixed">
+		<parent link="$(arg robot_name)_base_link"/>
+		<child link="$(arg robot_name)_top_chassis"/>
 	</joint>
-	<joint name="joint_left_wheel" type="continuous">
-		<parent link="base_link"/>
-		<child link="left_wheel"/>
+	<joint name="$(arg robot_name)_joint_left_wheel" type="continuous">
+		<parent link="$(arg robot_name)_base_link"/>
+		<child link="$(arg robot_name)_left_wheel"/>
 		<origin xyz="0 -.0728 0" rpy="0 0 0" />
 		<axis xyz="1 0 0" />
 	</joint>
-	<joint name="joint_right_wheel" type="continuous">
-		<parent link="base_link"/>
-		<child link="right_wheel"/>
+	<joint name="$(arg robot_name)_joint_right_wheel" type="continuous">
+		<parent link="$(arg robot_name)_base_link"/>
+		<child link="$(arg robot_name)_right_wheel"/>
 		<origin xyz="0 .0728 0" rpy="0 0 0" />
 		<axis xyz="1 0 0" />
 	</joint>
-	<joint name="joint_lidar" type="fixed">
-		<parent link="base_link" />
-		<child link="laser" />
+	<joint name="$(arg robot_name)_joint_lidar" type="fixed">
+		<parent link="$(arg robot_name)_base_link" />
+		<child link="$(arg robot_name)_laser" />
 		<origin xyz="-.05 0 0.0825" rpy="0 0 -1.5708" />
 	</joint>
-	<joint name="joint_imu" type="fixed">
-		<parent link="base_link" />
-		<child link="imu_link" />
+	<joint name="$(arg robot_name)_joint_imu" type="fixed">
+		<parent link="$(arg robot_name)_base_link" />
+		<child link="$(arg robot_name)_imu_link" />
 		<origin xyz="0 0 .05" rpy="0 0 0" />
 	</joint>
-	<joint name="joint_roadrunner" type="fixed">
-		<parent link="roadrunner" />
-		<child link="base_footprint" />
+	<joint name="$(arg robot_name)_joint_roadrunner" type="fixed">
+		<parent link="$(arg robot_name)_roadrunner" />
+		<child link="$(arg robot_name)_base_footprint" />
 		<origin xyz="0.0 0.0 -0.115" rpy="0 0 0" />
 	</joint>
