Commit message: SMB, all is working for 495, virtual nav, gazebo visualization. Not tested for IRL navigation.

File: usafabot_description/urdf/usafabot.gazebo.xacro (robot description, xacro)
@@ -112,5 +112,5 @@
         <alwaysOn>true</alwaysOn>
         <updateRate>0.0</updateRate>
-        <cameraName>camera</cameraName>
+        <cameraName>usb_cam</cameraName>
         <imageTopicName>image_raw</imageTopicName>
         <cameraInfoTopicName>camera_info</cameraInfoTopicName>

File: usafabot_description/urdf/usafabot.urdf.xacro (robot description, xacro)
@@ -215,6 +215,5 @@
     <parent link="base_link"/>
     <child link="imu_link"/>
-    <origin xyz="0 0 0.068" rpy="0 0 0"/>
-  </joint>
+    <origin xyz="0 0 0.068" rpy="0 0 -1.57"/>  </joint>
   <link name="imu_link"/>
 </robot>
