Commit message: Fixed color of LIDAR and camera for multi simulation.

File: usafabot_description/urdf/usafabot.gazebo_multi.xacro (robot description, xacro)
@@ -51,4 +51,7 @@
     <material>Gazebo/Black</material>
   </gazebo>
+  <gazebo reference="base_scan">
+    <material>Gazebo/FlatBlack</material>
+  </gazebo>
   <!-- LIDAR --><!--
   <gazebo reference="base_scan">
@@ -84,4 +87,7 @@
     </sensor>
   </gazebo>-->
+  <gazebo reference="camera_link">
+    <material>Gazebo/Black</material>
+  </gazebo>
   <!-- CAMERA --><!--
   <gazebo reference="camera_link">
